File: MCU Datalogger.kicad_sch (KiCad schematic)
At the start: 25 parts, among them U1 24LC1025, U2 DS1337S_, U3 24LC1025, U4 ATMEGA328P-AU, Y1 32.768 KHz, Y2 16MHz

Commit message: Footprints were added and fixed.
Parts:
- U2: footprint DS13375:DS13375 -> FOOTPRINTS:DS13375+
- U4: footprint ATMEGA:ATMEGA -> FOOTPRINTS:ATMEGA
Changed lines of the file:
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@@
 			)
 		)
-		(property "Footprint" "ATMEGA:ATMEGA"
+		(property "Footprint" "FOOTPRINTS:ATMEGA"
 			(at 213.36 64.77 0)
 			(effects
@@
 			)
 		)
-		(property "Footprint" "DS13375:DS13375"
+		(property "Footprint" "FOOTPRINTS:DS13375+"
 			(at 62.23 68.58 0)
 			(effects
