File: _autosave-MCU Datalogger.kicad_pcb (KiCad board)
At the start: 2 copper layers, 52.1 x 34.3 mm, 30 parts, among them J1 Conn_01x09_Pin, J2 Conn_01x04_Pin, J3 Conn_01x04_Pin, J4 Conn_02x03_Odd_Even, U1 24LC1025, U2 DS1337S_, U3 24LC1025, U4 ATMEGA328P-AU, Y1 32.768 KHz, Y2 16MHz

Commit message: Completed 2 layer.
Parts:
- added REF**: Symbol_GNU-Logo_SilkscreenTop, Symbol:Symbol_GNU-Logo_SilkscreenTop, B.Cu at (102.5, 74.0)
Other:
- board text added: "-2Mbit EEPROM -RTC -I2C, SPI, GPIO'S"

Commit message: 2 layer done.
Other:
- board text added: "0.0000 mm / 0.0000 mm"
- board text added: "0.3000 mm"
- board text added: "1.6000 mm"
- board text added: "2"
- board text added: "52.0650 mm x 34.2850 mm"
- board text added: "BOARD CHARACTERISTICS"
- board text added: "Board Thickness:"
- board text added: "Board overall dimensions:"
- board text added: "Castellated pads:"
- board text added: "Copper Finish:"
- board text added: "Copper Layer Count:"
- board text added: "Edge card connectors:"
- board text added: "Impedance Control:"
- board text added: "Min hole diameter:"
- board text added: "Min track/spacing:"
- board text added: "No"
- board text added: "None"
- board text added: "Plated Board Edge:"
