File: Connectors.kicad_sch (KiCad schematic)
At the start: 4 parts, among them J1 Conn_01x09_Pin, J2 Conn_01x04_Pin, J3 Conn_01x04_Pin, J4 Conn_02x03_Odd_Even

Commit message: Schec Missing.
Parts:
- renumbered J2 to J1, J1 to J2
Other:
- moved on the sheet: J1, J2, J3, J4
