File: MCU Datalogger.kicad_pcb (KiCad board)
At the start: 2 copper layers, 52.1 x 34.3 mm, 31 parts, among them J1 Conn_01x09_Pin, J2 Conn_01x04_Pin, J3 Conn_01x04_Pin, J4 Conn_02x03_Odd_Even, U1 24LC1025, U2 DS1337S_, U3 24LC1025, U4 ATMEGA328P-AU, Y1 32.768 KHz, Y2 16MHz

Commit message: Schec Missing.
Parts:
- moved REF** 2.75 mm to (102.7, 71.2)
- moved R7 0.28 mm to (121.0, 63.5)
- moved R4 0.25 mm to (121.0, 67.3), turned to 180 degrees
- moved U1 0.10 mm to (99.2, 68.6)
- turned C3 to 180 degrees
- turned C4 to 180 degrees
- turned R2 to 180 degrees
Routing:
- net /RESET: track 24.3 -> 78.6 mm, vias 2 -> 3
- net /SDA: track 69.6 -> 97.8 mm, vias 3 -> 5
- net /SCK: track 116.9 -> 138.6 mm, vias 9 -> 7
- net GND: track 91.0 -> 108.5 mm, vias 11 -> 16
- net /Vcc: track 138.6 -> 155.7 mm, vias 6 -> 9
- net /D7: track 18.8 -> 15.5 mm
- net Net-(U4-PB6): track 26.9 -> 23.9 mm
- net /D6: track 17.6 -> 15.5 mm
- net Net-(U4-PB7): track 23.1 -> 25.2 mm
- net Net-(U4-AREF): track 20.3 -> 18.7 mm
- net Net-(BT1-+): track 29.7 -> 28.2 mm, vias 1 -> 3
- net Net-(D2-K): track 5.19 -> 3.83 mm, vias 2 -> 0
- net /D5: track 17.1 -> 15.7 mm
- net Net-(U2-SQW/~INT): track 7.32 -> 6.27 mm
- net /D2: track 32.7 -> 31.8 mm
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Other:
- copper layers 2 -> 4
- board text removed: "0.0000 mm / 0.0000 mm"
- board text removed: "0.3000 mm"
- board text removed: "1.6000 mm"
- board text removed: "2"
- board text removed: "52.0650 mm x 34.2850 mm"
- board text removed: "BOARD CHARACTERISTICS"
- board text removed: "Board Thickness:"
- board text removed: "Board overall dimensions:"
- board text removed: "Castellated pads:"
- board text removed: "Copper Finish:"
- board text removed: "Copper Layer Count:"
- board text removed: "Edge card connectors:"
- board text removed: "Impedance Control:"
- board text removed: "Min hole diameter:"
- board text removed: "Min track/spacing:"
- board text removed: "No"
- board text removed: "None"
- board text removed: "Plated Board Edge:"
